File: bike-headlamp/bike-headlamp.kicad_pcb (KiCad board)
At the start: 2 copper layers, 9 parts, among them J1 HARNESS, J2 HEADSET, J3 LED1, J4 LED2, SW1 FRONT, SW2 BACK, U1 Digispark, U2 MiniPuck, U3 MiniPuck

Commit message: finalized board?
Parts:
- removed J2: HEADSET, Pin_Headers:Pin_Header_Straight_1x04_Pitch2.54mm
- removed J3: LED1, Pin_Headers:Pin_Header_Straight_1x02_Pitch2.54mm
- added J5: LED2, Pin_Headers:Pin_Header_Straight_1x02_Pitch2.54mm, F.Cu at (142.3, 64.5)
- J1: value HARNESS -> HARNESS5-8; footprint Pin_Headers:Pin_Header_Straight_1x08_Pitch2.54mm -> Pin_Headers:Pin_Header_Straight_1x04_Pitch2.54mm
- J4: value LED2 -> LED1
- SW1, SW2: footprint Buttons_Switches_SMD:SW_SPST_PTS810 -> Pin_Headers:Pin_Header_Straight_1x02_Pitch2.54mm
- U3: moved to B.Cu
- moved SW2 74.2 mm to (136.4, 71.6), turned to 270 degrees
- moved U2 65.1 mm to (145.9, 71.9), turned to 180 degrees
- moved J1 57.2 mm to (128.0, 61.8)
- moved U3 51.5 mm to (128.1, 74.1)
- moved U1 39.8 mm to (130.8, 67.7), turned to 270 degrees
- moved SW1 35.5 mm to (136.4, 68.8), turned to 270 degrees
- moved J4 30.1 mm to (136.3, 61.9), turned to 270 degrees
Connections:
- net Net-(SW1-Pad2) renamed /SW-FRONT
- net Net-(SW2-Pad2) renamed /SW-BACK
- net Net-(U1-Pad2) renamed /LED1-PWM
- net Net-(U1-Pad5) renamed /LED2-PWM
- J1 pad 1: Net-(J1-Pad1) -> /SCL
- J1 pad 2: Net-(J1-Pad2) -> /SDA
- J1 pad 3: Net-(J1-Pad3) -> +12V
- J1 pad 4: Net-(J1-Pad4) -> GNDREF
- J4 pad 1: Net-(J4-Pad1) -> /LED1+
- J4 pad 2: Net-(J4-Pad2) -> /LED1-
- U1 pad 1: Net-(J1-Pad6) -> /SDA
- U1 pad 3: Net-(J1-Pad5) -> /SCL
- U2 pad 4: Net-(J3-Pad1) -> /LED1+
- U2 pad 5: Net-(J3-Pad2) -> /LED1-
- U3 pad 4: Net-(J4-Pad1) -> /LED2+
- U3 pad 5: Net-(J4-Pad2) -> /LED2-
Routing:
- net /LED2-PWM: track 0.00 -> 16.1 mm
- net /LED1-PWM: track 0.00 -> 9.03 mm
- net /LED1-: track 0.00 -> 6.71 mm
- net /SCL: track 0.00 -> 5.78 mm
- net /LED1+: track 0.00 -> 4.17 mm
- net /SDA: track 0.00 -> 4.15 mm
- net /SW-BACK: track 0.00 -> 4.13 mm
- net /LED2+: track 0.00 -> 3.65 mm
- net /LED2-: track 0.00 -> 3.50 mm
- net /SW-FRONT: track 0.00 -> 3.12 mm
- added copper zone on F.Cu, net +12V
- added copper zone on B.Cu, net GNDREF
Other:
- board outline added: 20.1 x 19.1 mm
- net class Default: clearance 0.2 -> 0.1524; trace_width 0.25 -> 0.1524; via_dia 0.8 -> 0.508; via_drill 0.4 -> 0.254
- net class LED-Power added: clearance 0.1524, trace_width 0.2032, via_dia 0.508, via_drill 0.254
- rule trace_clearance: 0.2 -> 0.1524
- rule trace_min: 0.2 -> 0.1524
- rule via_min_drill: 0.3 -> 0.254
- rule via_min_size: 0.4 -> 0.508
