File: bike-headlamp-controller-pcb/bike-headlamp-controller-pcb/bike-headlamp-controller-pcb.sch (KiCad schematic (older format))
At the start: 23 parts, among them J1 12V in, J2 i2c_hv, J3 LED, J4 USB_B_Micro, J5 switch, U1 P82B96, U2 MC78M05_TO252, U3 MiniPuck, U4 ATTINY85-20SU

Commit message: finished initial draft of pcb
Parts:
- removed C1: 0.33uF, Capacitor_SMD:C_2220_5650Metric_Pad2.02x5.50mm_HandSolder, symbol Device:CP1
- removed C2: 4.7uF, Capacitor_SMD:C_0805_2012Metric_Pad1.15x1.50mm_HandSolder, symbol Device:C
- removed D3, D4: 3.6V Zener, symbol Device:D_Zener
- removed J4: USB_B_Micro, SW-Hirose:ZX62D-B-5PA8(30), symbol Connector_Specialized:USB_B_Micro
- removed R5: 1k5Ω, symbol Device:R
- removed R6, R7: 66.5Ω, symbol Device:R
- removed U2: MC78M05_TO252, Package_TO_SOT_SMD:TO-252-2, symbol Regulator_Linear:MC78M05_TO252
- added C2, C3: 22uF, Capacitor_SMD:C_0805_2012Metric, symbol Device:C_Small
- added C4: 10uF, Capacitor_SMD:C_0603_1608Metric, symbol Device:C_Small
- added J4: ISC Header, SW-test-pads:isc-pogo-pins, symbol Connector_Generic:Conn_02x03_Odd_Even
- added U3: LMZM23600V5SILT, SW-Texas:SIL0010A, symbol SW-Texas:LMZM23600V5SILT
- J1: renamed from J2; footprint SW-4UCON:JST-2pole-RA -> SW-JST:JST-2pole
- J2: renamed from J1; footprint (none) -> SW-JST:JST-2pole
- J3, J5: footprint (none) -> SW-JST:JST-2pole
- R1, R2, R3, R4: footprint (none) -> Resistor_SMD:R_0402_1005Metric
- renumbered C3 to C1, U3 to U2
Connections:
- net labels added: +5V_MCU, MISO, MOSI, SCK, ~RESET
- net labels removed: USB_D+, USB_D-, VBUS
- wire segments 122 -> 121
- no-connect marks 1 -> 2
Other:
- note added: "1 - MISO\n2 - VCC\n3 - SCK\n4 - MOSI\n5 - RESET\n6 - GND"
- note added: "Need external VCC to program"
- note added: "Programming Voltage\nor board voltage can power\nMCU but programming\nvoltage cannot backfeed into \nremainder of circuit"
